File: roomba_main_pcb_v1.brd (EAGLE design)
At the start: 37 x 40 mm, 14 parts, among them J1 J25MM

Commit message: 1.0
Parts:
- turned JP4 to 270 degrees
Connections:
- net GND: now also JP1.4; no longer JP1.1
- net N$12: now also JP1.3; no longer JP1.4
- net N$13: now also JP1.1; no longer JP1.2
- net N$15: now also JP1.2; no longer JP1.3
Routing:
- net N$12: track 46.0 -> 51.4 mm
- net N$15: track 32.3 -> 27.3 mm
- net N$13: track 26.9 -> 31.5 mm
Changed lines of the file:
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@@
 <attribute name="VALUE" x="17.715" y="3.83" size="1.27" layer="27" rot="R270"/>
 </element>
-<element name="JP4" library="pinhead" library_urn="urn:adsk.eagle:library:325" package="1X02" package3d_urn="urn:adsk.eagle:package:22435/2" value="" x="-6" y="-1" smashed="yes" rot="R90">
-<attribute name="NAME" x="-7.8288" y="-3.6162" size="1.27" layer="25" ratio="10" rot="R90"/>
-<attribute name="POPULARITY" value="98" x="-6" y="-1" size="1.778" layer="27" rot="R90" display="off"/>
-<attribute name="VALUE" x="-2.825" y="-3.54" size="1.27" layer="27" rot="R90"/>
+<element name="JP4" library="pinhead" library_urn="urn:adsk.eagle:library:325" package="1X02" package3d_urn="urn:adsk.eagle:package:22435/2" value="" x="-6" y="-1" smashed="yes" rot="R270">
+<attribute name="NAME" x="-4.1712" y="1.6162" size="1.27" layer="25" ratio="10" rot="R270"/>
+<attribute name="POPULARITY" value="98" x="-6" y="-1" size="1.778" layer="27" rot="R270" display="off"/>
+<attribute name="VALUE" x="-9.175" y="1.54" size="1.27" layer="27" rot="R270"/>
 </element>
 </elements>
@@
 <contactref element="U$1" pad="OUT-.1"/>
 <contactref element="U$1" pad="IN-.1"/>
-<contactref element="JP1" pad="1"/>
 <contactref element="JP3" pad="1"/>
+<contactref element="JP1" pad="4"/>
 </signal>
 <signal name="N$3">
@@
 </signal>
 <signal name="N$12">
-<contactref element="JP1" pad="4"/>
-<wire x1="-0.51" y1="25.38" x2="-0.51" y2="26.88" width="1" layer="16"/>
-<wire x1="-0.51" y1="25.38" x2="-2.01" y2="23.88" width="1" layer="16"/>
-<wire x1="-2.01" y1="23.88" x2="-2.01" y2="8.21" width="1" layer="16"/>
 <contactref element="JP3" pad="2"/>
-<wire x1="20.89" y1="-0.98" x2="7.18" y2="-0.98" width="1" layer="16"/>
-<wire x1="7.18" y1="-0.98" x2="-2.01" y2="8.21" width="1" layer="16"/>
+<wire x1="20.89" y1="-0.98" x2="-0.32" y2="-0.98" width="1" layer="16"/>
+<wire x1="-0.32" y1="-0.98" x2="-4.51" y2="3.21" width="1" layer="16"/>
+<contactref element="JP1" pad="3"/>
+<wire x1="-3.05" y1="26.88" x2="-3.05" y2="24.84" width="1" layer="16"/>
+<wire x1="-3.05" y1="24.84" x2="-4.51" y2="23.38" width="1" layer="16"/>
+<wire x1="-4.51" y1="23.38" x2="-4.51" y2="3.21" width="1" layer="16"/>
 </signal>
 <signal name="N$13">
-<contactref element="JP1" pad="2"/>
 <contactref element="JP4" pad="2"/>
-<wire x1="-6" y1="0.27" x2="-6.2" y2="0.47" width="1.5" layer="16"/>
-<wire x1="-5.59" y1="26.88" x2="-5.59" y2="25.88" width="1.5" layer="16"/>
-<wire x1="-5.59" y1="25.88" x2="-6.2" y2="25.27" width="1.5" layer="16"/>
-<wire x1="-6.2" y1="25.27" x2="-6.2" y2="0.47" width="1.5" layer="16"/>
+<contactref element="JP1" pad="1"/>
+<wire x1="-9.09" y1="25.92" x2="-8.13" y2="26.88" width="1.5" layer="16"/>
+<wire x1="-6" y1="-2.27" x2="-7.23" y2="-2.27" width="1.5" layer="16"/>
+<wire x1="-7.23" y1="-2.27" x2="-9.09" y2="-0.41" width="1.5" layer="16"/>
+<wire x1="-9.09" y1="-0.41" x2="-9.09" y2="25.92" width="1.5" layer="16"/>
 </signal>
 <signal name="N$14">
@@
 </signal>
 <signal name="N$15">
-<contactref element="JP1" pad="3"/>
 <contactref element="JP4" pad="1"/>
-<wire x1="-3.05" y1="26.88" x2="-3.05" y2="25.38" width="1.5" layer="16"/>
-<wire x1="-3.05" y1="25.38" x2="-4.05" y2="24.38" width="1.5" layer="16"/>
-<wire x1="-4.05" y1="24.38" x2="-4.05" y2="2.55" width="1.5" layer="16"/>
-<wire x1="-3" y1="1.5" x2="-3" y2="-1" width="1.5" layer="16"/>
-<wire x1="-3" y1="-1" x2="-4.27" y2="-2.27" width="1.5" layer="16"/>
-<wire x1="-6" y1="-2.27" x2="-4.27" y2="-2.27" width="1.5" layer="16"/>
-<wire x1="-4.05" y1="2.55" x2="-3" y2="1.5" width="1.5" layer="16"/>
+<contactref element="JP1" pad="2"/>
+<wire x1="-5.59" y1="26.88" x2="-5.59" y2="25.38" width="1.5" layer="16"/>
+<wire x1="-5.59" y1="25.38" x2="-6.59" y2="24.38" width="1.5" layer="16"/>
+<wire x1="-6.59" y1="24.38" x2="-6.59" y2="1.09" width="1.5" layer="16"/>
+<wire x1="-6" y1="0.5" x2="-6" y2="0.27" width="1.5" layer="16"/>
+<wire x1="-6.59" y1="1.09" x2="-6" y2="0.5" width="1.5" layer="16"/>
 </signal>
 </signals>

Commit message: 1.1
Parts:
- renumbered JP3 to LED_DRIVER_IN, JP4 to LED_DRIVER_OUT, U$3 to ROOMBA_PORT
Connections:
- net N$1 renamed GPIO_23
- net N$10 renamed 5V_RPI
- net N$12 renamed GPIO_18
- net N$13 renamed PWR_LED
- net N$14 renamed GPIO_14
- net N$15 renamed GND_LED
- net N$3 renamed GPIO_15
Changed lines of the file:
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@@
 <attribute name="VALUE" x="24.193" y="16.644" size="1.27" layer="28" rot="MR270"/>
 </element>
-<element name="U$3" library="M_wifi" package="PIN-7" value="7_PIN" x="9.9" y="15.89" smashed="yes" rot="R180"/>
+<element name="ROOMBA_PORT" library="M_wifi" package="PIN-7" value="7_PIN" x="9.9" y="15.89" smashed="yes" rot="R180"/>
 <element name="R4" library="rcl" library_urn="urn:adsk.eagle:library:334" package="M1206" package3d_urn="urn:adsk.eagle:package:23566/2" value="390" x="9.44" y="10.38" smashed="yes" rot="MR0">
 <attribute name="NAME" x="10.71" y="11.65" size="1.27" layer="26" rot="MR0"/>
@@
 <attribute name="VALUE" x="15.38" y="15.85" size="0.02" layer="27" rot="R270"/>
 </element>
-<element name="JP3" library="pinhead" library_urn="urn:adsk.eagle:library:325" package="1X03" package3d_urn="urn:adsk.eagle:package:22458/2" value="" x="20.89" y="-0.98" smashed="yes" rot="R270">
+<element name="LED_DRIVER_IN" library="pinhead" library_urn="urn:adsk.eagle:library:325" package="1X03" package3d_urn="urn:adsk.eagle:package:22458/2" value="" x="20.89" y="-0.98" smashed="yes" rot="R270">
 <attribute name="NAME" x="22.7188" y="3.9062" size="1.27" layer="25" ratio="10" rot="R270"/>
 <attribute name="POPULARITY" value="92" x="20.89" y="0.02" size="1.778" layer="27" rot="R270" display="off"/>
 <attribute name="VALUE" x="17.715" y="3.83" size="1.27" layer="27" rot="R270"/>
 </element>
-<element name="JP4" library="pinhead" library_urn="urn:adsk.eagle:library:325" package="1X02" package3d_urn="urn:adsk.eagle:package:22435/2" value="" x="-6" y="-1" smashed="yes" rot="R270">
+<element name="LED_DRIVER_OUT" library="pinhead" library_urn="urn:adsk.eagle:library:325" package="1X02" package3d_urn="urn:adsk.eagle:package:22435/2" value="" x="-6" y="-1" smashed="yes" rot="R270">
 <attribute name="NAME" x="-4.1712" y="1.6162" size="1.27" layer="25" ratio="10" rot="R270"/>
 <attribute name="POPULARITY" value="98" x="-6" y="-1" size="1.778" layer="27" rot="R270" display="off"/>
@@
 </polygon>
 <contactref element="D3" pad="A"/>
-<contactref element="U$3" pad="GND_1"/>
+<contactref element="ROOMBA_PORT" pad="GND_1"/>
 <contactref element="U$1" pad="OUT-.1"/>
 <contactref element="U$1" pad="IN-.1"/>
-<contactref element="JP3" pad="1"/>
+<contactref element="LED_DRIVER_IN" pad="1"/>
 <contactref element="JP1" pad="4"/>
 </signal>
-<signal name="N$3">
+<signal name="GPIO_15">
 <contactref element="D2" pad="C"/>
 <contactref element="R2" pad="1"/>
@@
 <wire x1="2" y1="17.5" x2="2" y2="16.5" width="1" layer="16"/>
 </signal>
-<signal name="N$1">
+<signal name="GPIO_23">
 <contactref element="R4" pad="1"/>
 <contactref element="D3" pad="C"/>
@@
 </signal>
 <signal name="+18V">
-<contactref element="U$3" pad="VPWR_1"/>
+<contactref element="ROOMBA_PORT" pad="VPWR_1"/>
 <contactref element="JP1" pad="9"/>
 <wire x1="12.19" y1="26.88" x2="12.19" y2="20.08" width="1.5" layer="16"/>
@@
 </signal>
 <signal name="N$5">
-<contactref element="U$3" pad="DD"/>
+<contactref element="ROOMBA_PORT" pad="DD"/>
 <contactref element="R4" pad="2"/>
 <wire x1="7.9" y1="13.99" x2="7.77" y2="13.86" width="1" layer="16"/>
@@
 <signal name="N$7">
 <contactref element="R3" pad="2"/>
-<contactref element="U$3" pad="RX"/>
+<contactref element="ROOMBA_PORT" pad="RX"/>
 <wire x1="5" y1="16.66" x2="5.06946875" y2="16.627746875" width="0.254" layer="16"/>
 <wire x1="5.06946875" y1="16.627746875" x2="4.46" y2="16.4" width="0.254" layer="16"/>
@@
 <signal name="N$9">
 <contactref element="R2" pad="2"/>
-<contactref element="U$3" pad="TX"/>
+<contactref element="ROOMBA_PORT" pad="TX"/>
 <wire x1="15.9" y1="17.39" x2="13.4" y2="17.39" width="1" layer="16"/>
 <wire x1="13.4" y1="17.39" x2="12.4" y2="16.39" width="1" layer="16"/>
 <wire x1="15.9" y1="17.39" x2="15.73" y2="17.37" width="0" layer="19" extent="16-16"/>
 </signal>
-<signal name="N$10">
+<signal name="5V_RPI">
 <contactref element="U$1" pad="OUT+.2"/>
 <contactref element="JP1" pad="5"/>
@@
 <signal name="N$6">
 <contactref element="J1" pad="2"/>
-<contactref element="JP3" pad="3"/>
+<contactref element="LED_DRIVER_IN" pad="3"/>
 <wire x1="20.77" y1="-3.4" x2="15.93" y2="-3.4" width="1.5" layer="16"/>
 <wire x1="15.88" y1="-3.35" x2="15.93" y2="-3.4" width="1.5" layer="16"/>
 <wire x1="20.89" y1="-3.52" x2="20.77" y2="-3.4" width="1.5" layer="16"/>
 </signal>
-<signal name="N$12">
-<contactref element="JP3" pad="2"/>
+<signal name="GPIO_18">
+<contactref element="LED_DRIVER_IN" pad="2"/>
 <wire x1="20.89" y1="-0.98" x2="-0.32" y2="-0.98" width="1" layer="16"/>
 <wire x1="-0.32" y1="-0.98" x2="-4.51" y2="3.21" width="1" layer="16"/>
@@
 <wire x1="-4.51" y1="23.38" x2="-4.51" y2="3.21" width="1" layer="16"/>
 </signal>
-<signal name="N$13">
-<contactref element="JP4" pad="2"/>
+<signal name="PWR_LED">
+<contactref element="LED_DRIVER_OUT" pad="2"/>
 <contactref element="JP1" pad="1"/>
 <wire x1="-9.09" y1="25.92" x2="-8.13" y2="26.88" width="1.5" layer="16"/>
@@
 <wire x1="-9.09" y1="-0.41" x2="-9.09" y2="25.92" width="1.5" layer="16"/>
 </signal>
-<signal name="N$14">
+<signal name="GPIO_14">
 <contactref element="JP1" pad="6"/>
 <contactref element="R1" pad="1"/>
@@
 <wire x1="5.66" y1="24.68" x2="5.66" y2="23.18" width="1" layer="16"/>
 </signal>
-<signal name="N$15">
-<contactref element="JP4" pad="1"/>
+<signal name="GND_LED">
+<contactref element="LED_DRIVER_OUT" pad="1"/>
 <contactref element="JP1" pad="2"/>
 <wire x1="-5.59" y1="26.88" x2="-5.59" y2="25.38" width="1.5" layer="16"/>
