File: roomba_main_pcb_v1.sch (EAGLE design)
At the start: 14 parts, among them J1 J25MM

Commit message: 1.0
Connections:
- net GND: now also JP1.4; no longer JP1.1
- net N$12: now also JP1.3; no longer JP1.4
- net N$13: now also JP1.1; no longer JP1.2
- net N$15: now also JP1.2; no longer JP1.3
Changed lines of the file:
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@@
 <attribute name="VALUE" x="31.75" y="17.78" size="1.778" layer="96"/>
 </instance>
-<instance part="SUPPLY3" gate="GND" x="25.4" y="45.72" smashed="yes" rot="R180">
-<attribute name="VALUE" x="27.305" y="48.895" size="1.778" layer="96" rot="R180"/>
+<instance part="SUPPLY3" gate="GND" x="17.78" y="30.48" smashed="yes" rot="R270">
+<attribute name="VALUE" x="14.605" y="32.385" size="1.778" layer="96" rot="R270"/>
 </instance>
 <instance part="U$1" gate="G$1" x="-7.62" y="17.78" smashed="yes" rot="R180">
@@
 </segment>
 <segment>
-<pinref part="SUPPLY3" gate="GND" pin="GND"/>
-<wire x1="25.4" y1="43.18" x2="35.56" y2="43.18" width="0.1524" layer="91"/>
-<wire x1="35.56" y1="43.18" x2="35.56" y2="38.1" width="0.1524" layer="91"/>
-<junction x="25.4" y="43.18"/>
-<pinref part="JP1" gate="A" pin="1"/>
-<junction x="35.56" y="38.1"/>
-</segment>
-<segment>
 <pinref part="U$1" gate="G$1" pin="OUT-.1"/>
 <pinref part="SUPPLY1" gate="GND" pin="GND"/>
@@
 <wire x1="38.1" y1="-12.7" x2="30.48" y2="-12.7" width="0.1524" layer="91"/>
 <junction x="38.1" y="-12.7"/>
+</segment>
+<segment>
+<pinref part="JP1" gate="A" pin="4"/>
+<pinref part="SUPPLY3" gate="GND" pin="GND"/>
+<wire x1="35.56" y1="30.48" x2="20.32" y2="30.48" width="0.1524" layer="91"/>
 </segment>
 </net>
@@
 <wire x1="2.54" y1="33.02" x2="2.54" y2="-10.16" width="0.1524" layer="91"/>
 <wire x1="2.54" y1="-10.16" x2="38.1" y2="-10.16" width="0.1524" layer="91"/>
-<pinref part="JP1" gate="A" pin="4"/>
-<wire x1="35.56" y1="30.48" x2="10.16" y2="30.48" width="0.1524" layer="91"/>
-<wire x1="10.16" y1="30.48" x2="10.16" y2="33.02" width="0.1524" layer="91"/>
-<wire x1="10.16" y1="33.02" x2="2.54" y2="33.02" width="0.1524" layer="91"/>
-<junction x="35.56" y="30.48"/>
 <pinref part="JP3" gate="A" pin="2"/>
 <junction x="38.1" y="-10.16"/>
+<pinref part="JP1" gate="A" pin="3"/>
+<wire x1="35.56" y1="33.02" x2="2.54" y2="33.02" width="0.1524" layer="91"/>
 </segment>
 </net>
 <net name="N$13" class="0">
 <segment>
-<pinref part="JP1" gate="A" pin="2"/>
 <pinref part="JP4" gate="G$1" pin="2"/>
-<wire x1="35.56" y1="35.56" x2="17.78" y2="35.56" width="0.1524" layer="91"/>
-<wire x1="17.78" y1="35.56" x2="17.78" y2="43.18" width="0.1524" layer="91"/>
-<junction x="35.56" y="35.56"/>
 <junction x="17.78" y="43.18"/>
+<pinref part="JP1" gate="A" pin="1"/>
+<wire x1="17.78" y1="38.1" x2="17.78" y2="43.18" width="0.1524" layer="91"/>
+<wire x1="35.56" y1="38.1" x2="17.78" y2="38.1" width="0.1524" layer="91"/>
 </segment>
 </net>
@@
 <net name="N$15" class="0">
 <segment>
-<pinref part="JP1" gate="A" pin="3"/>
-<wire x1="35.56" y1="33.02" x2="15.24" y2="33.02" width="0.1524" layer="91"/>
-<wire x1="15.24" y1="33.02" x2="15.24" y2="43.18" width="0.1524" layer="91"/>
 <pinref part="JP4" gate="G$1" pin="1"/>
 <junction x="15.24" y="43.18"/>
-</segment>
-</net>
+<pinref part="JP1" gate="A" pin="2"/>
+<wire x1="15.24" y1="35.56" x2="15.24" y2="43.18" width="0.1524" layer="91"/>
+<wire x1="35.56" y1="35.56" x2="15.24" y2="35.56" width="0.1524" layer="91"/>
+</segment>
+</net>

Commit message: 1.1
Parts:
- removed JP3: (no value), pinhead:PINHD-1X3
- removed JP4: (no value), pinhead:PINHD-1X2
- removed U$3: 7_PIN, M_wifi:7_PIN
- added LED_DRIVER_IN: (no value), pinhead:PINHD-1X3
- added LED_DRIVER_OUT: (no value), pinhead:PINHD-1X2
- added ROOMBA_PORT: 7_PIN, M_wifi:7_PIN
Connections:
- net N$1 renamed GPIO_23
- net N$10 renamed 5V_RPI
- net N$14 renamed GPIO_14
- net N$3 renamed GPIO_15
- removed net N$12: JP1.3, JP3.2
- removed net N$13: JP1.1, JP4.2
- removed net N$15: JP1.2, JP4.1
- new net GND_LED: JP1.2, LED_DRIVER_OUT.1
- new net GPIO_18: JP1.3, LED_DRIVER_IN.2
- new net PWR_LED: JP1.1, LED_DRIVER_OUT.2
- net +18V: now also ROOMBA_PORT.V_PWR1; no longer U$3.V_PWR1
- net GND: now also LED_DRIVER_IN.1, ROOMBA_PORT.GND_1; no longer JP3.1, U$3.GND_1
- net N$5: now also ROOMBA_PORT.DD; no longer U$3.DD
- net N$6: now also LED_DRIVER_IN.3; no longer JP3.3
- net N$7: now also ROOMBA_PORT.RX; no longer U$3.RX
- net N$9: now also ROOMBA_PORT.TX; no longer U$3.TX
Other:
- moved on the sheet: D1, D2, D3, J1, R1, R2, R3, R4, R5, U$1
