File: pcb/roomba_led_pcb_v1.brd (EAGLE design)
At the start: 47.5 x 35.5 mm, 3 parts

Commit message: 1.1
Parts:
- moved JP5 4.67 mm to (-17.0, 15.0)
- moved JP3 2.92 mm to (-15.0, 5.00)
- moved JP4 1.50 mm to (-2.94, 8.84)
Routing:
- net N$2: track 20.6 -> 23.3 mm
- net N$1: track 8.42 -> 10.9 mm
- added copper zone on layer 16, net GND
- removed copper zone on layer 1, net GND
Changed lines of the file:
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@@
 <hole x="-18.5" y="-2" drill="3"/>
 <hole x="-18.5" y="21.5" drill="3"/>
-<rectangle x1="11.5" y1="5.5" x2="20.5" y2="14.5" layer="1"/>
-<rectangle x1="3.5" y1="5.5" x2="11.5" y2="14.5" layer="1"/>
-<rectangle x1="3.5" y1="3.5" x2="8.5" y2="5.5" layer="1"/>
-<hole x="-12.5" y="9.83" drill="6"/>
+<rectangle x1="11.5" y1="5.5" x2="20.5" y2="14.5" layer="16"/>
+<rectangle x1="3.5" y1="5.5" x2="11.5" y2="14.5" layer="16"/>
+<rectangle x1="3.5" y1="3.5" x2="8.5" y2="5.5" layer="16"/>
+<hole x="-16.01" y="9.99" drill="6"/>
 </plain>
 <attributes>
@@
 </autorouter>
 <elements>
-<element name="JP4" library="pinhead" library_urn="urn:adsk.eagle:library:325" package="1X02/90" package3d_urn="urn:adsk.eagle:package:22437/2" value="" x="-2.94" y="7.34" smashed="yes">
-<attribute name="NAME" x="-5.5562" y="9.1688" size="1.27" layer="25" ratio="10"/>
-<attribute name="POPULARITY" value="24" x="-2.94" y="7.34" size="1.778" layer="27" display="off"/>
-<attribute name="VALUE" x="-5.48" y="4.165" size="1.27" layer="27"/>
+<element name="JP4" library="pinhead" library_urn="urn:adsk.eagle:library:325" package="1X02/90" package3d_urn="urn:adsk.eagle:package:22437/2" value="" x="-2.94" y="8.84" smashed="yes">
+<attribute name="NAME" x="-5.5562" y="10.6688" size="1.27" layer="25" ratio="10"/>
+<attribute name="POPULARITY" value="24" x="-2.94" y="8.84" size="1.778" layer="27" display="off"/>
+<attribute name="VALUE" x="-5.48" y="5.665" size="1.27" layer="27"/>
 </element>
-<element name="JP3" library="pinhead_new" package="1X01" package3d_urn="urn:adsk.eagle:package:22485/2" value="" x="-12.5" y="3.5" smashed="yes">
-<attribute name="NAME" x="-13.3462" y="0.3288" size="1.27" layer="25" ratio="10"/>
-<attribute name="POPULARITY" value="64" x="-12.5" y="3.5" size="1.778" layer="27" display="off"/>
-<attribute name="VALUE" x="-13.77" y="0.325" size="1.27" layer="27"/>
+<element name="JP3" library="pinhead_new" package="1X01" package3d_urn="urn:adsk.eagle:package:22485/2" value="" x="-15" y="5" smashed="yes">
+<attribute name="NAME" x="-15.8462" y="1.8288" size="1.27" layer="25" ratio="10"/>
+<attribute name="POPULARITY" value="64" x="-15" y="5" size="1.778" layer="27" display="off"/>
+<attribute name="VALUE" x="-16.27" y="1.825" size="1.27" layer="27"/>
 </element>
-<element name="JP5" library="pinhead_new" package="1X01" package3d_urn="urn:adsk.eagle:package:22485/2" value="" x="-12.46" y="16.16" smashed="yes">
-<attribute name="NAME" x="-13.8062" y="17.9888" size="1.27" layer="25" ratio="10"/>
-<attribute name="POPULARITY" value="64" x="-12.46" y="16.16" size="1.778" layer="27" display="off"/>
-<attribute name="VALUE" x="-13.73" y="12.985" size="1.27" layer="27"/>
+<element name="JP5" library="pinhead_new" package="1X01" package3d_urn="urn:adsk.eagle:package:22485/2" value="" x="-16.99" y="15.03" smashed="yes">
+<attribute name="NAME" x="-18.3362" y="16.8588" size="1.27" layer="25" ratio="10"/>
+<attribute name="POPULARITY" value="64" x="-16.99" y="15.03" size="1.778" layer="27" display="off"/>
+<attribute name="VALUE" x="-18.26" y="11.855" size="1.27" layer="27"/>
 </element>
 </elements>
 <signals>
 <signal name="GND">
-<polygon width="0.1" layer="1" isolate="0.6" thermals="no">
+<polygon width="0.1" layer="16" isolate="0.6" thermals="no">
 <vertex x="26.3" y="30.69"/>
 <vertex x="-21.7" y="30.69"/>
@@
 <signal name="N$2">
 <contactref element="JP4" pad="2"/>
-<wire x1="-1.67" y1="3.53" x2="-1.67" y2="11.504" width="1.5" layer="1"/>
-<wire x1="-1.67" y1="11.504" x2="-6.27" y2="16.104" width="1.5" layer="1"/>
-<wire x1="-6.27" y1="16.104" x2="-12.396" y2="16.104" width="1.5" layer="1"/>
+<wire x1="-1.67" y1="5.03" x2="-1.67" y2="11.504" width="1.5" layer="16"/>
+<wire x1="-1.67" y1="11.504" x2="-5.17" y2="15.004" width="1.5" layer="16"/>
+<wire x1="-5.17" y1="15.004" x2="-17.016" y2="15.004" width="1.5" layer="16"/>
 <contactref element="JP5" pad="1"/>
-<wire x1="-12.396" y1="16.104" x2="-12.46" y2="16.16" width="0" layer="19" extent="1-1"/>
+<wire x1="-16.99" y1="15.03" x2="-17.016" y2="15.004" width="0" layer="19" extent="16-16"/>
 </signal>
 <signal name="N$1">
 <contactref element="JP4" pad="1"/>
-<wire x1="-4.25" y1="3.49" x2="-4.24" y2="3.5" width="1.5" layer="16"/>
-<wire x1="-4.24" y1="3.5" x2="-4.21" y2="3.53" width="1.5" layer="16"/>
-<wire x1="-4.21" y1="3.53" x2="-4.24" y2="3.5" width="1.5" layer="16"/>
-<wire x1="-4.24" y1="3.5" x2="-12.56" y2="3.5" width="1.5" layer="1"/>
+<wire x1="-4.25" y1="4.99" x2="-4.21" y2="5.03" width="1.5" layer="16"/>
+<wire x1="-4.21" y1="5.03" x2="-4.24" y2="5" width="1.5" layer="16"/>
+<wire x1="-4.24" y1="5" x2="-15.06" y2="5" width="1.5" layer="16"/>
 <contactref element="JP3" pad="1"/>
-<wire x1="-12.56" y1="3.5" x2="-12.5" y2="3.5" width="0" layer="19" extent="1-1"/>
-<wire x1="-4.25" y1="3.49" x2="-4.24" y2="3.5" width="0" layer="19" extent="1-16"/>
+<wire x1="-15.06" y1="5" x2="-15" y2="5" width="0" layer="19" extent="16-16"/>
 </signal>
 </signals>
